Commit message: Removed coupler from gripper

File: robotiq_description/urdf/robotiq_hande_macro.urdf.xacro (robot description, xacro)
@@ -20,14 +20,8 @@
         gripper_closed_position:=0.025">
         <!-- Robotiq Hand-E specs -->
-        <!--  + Height added by the IO coupler: 11.0mm -->
         <!--  + Height added by the Hand-E body: 99.0mm -->
         <!--  + Finger protrusion above body: 46.5mm -->
-        <xacro:property name="coupler_height" value="0.011" />
-        <xacro:property name="coupler_shell_height" value="0.0169" />
-        <xacro:property name="coupler_parent_cutoff" value="0.003" />
-        <xacro:property name="coupler_hande_cutoff" value="0.0029" />
         <xacro:property name="hande_height" value="0.099" />
         <xacro:property name="hande_radius" value="0.0375" />
-        <xacro:property name="coupler_mass" value="0.119" />
         <!-- ros2 control include -->
         <xacro:include filename="$(find robotiq_description)/urdf/hande.ros2_control.xacro" />
@@ -49,38 +43,9 @@
                 gripper_closed_position="${gripper_closed_position}"/>
         </xacro:if>
-        <!-- IO coupler -->
-        <joint name="${prefix}robotiq_hande_coupler_joint" type="fixed">
-            <parent link="${parent}" />
-            <child link="${prefix}robotiq_hande_coupler" />
-            <xacro:insert_block name="origin" />
-        </joint>
-        <link name="${prefix}robotiq_hande_coupler">
-            <visual>
-                <geometry>
-                    <mesh filename="package://robotiq_description/meshes/visual/hande/io_coupler.dae" />
-                </geometry>
-            </visual>
-            <collision>
-                <origin xyz="0 0 ${coupler_shell_height/2 - coupler_parent_cutoff}" rpy="0 0 0" />
-                <geometry>
-                    <cylinder length="${coupler_shell_height}" radius="${hande_radius + 0.001}" />
-                </geometry>
-            </collision>
-            <inertial>
-                <origin xyz="0 0 ${coupler_shell_height/2 - coupler_parent_cutoff}" rpy="0 0 0" />
-                <mass value="${coupler_mass}" />
-                <inertia
-                    ixx="${0.0833333 * coupler_mass * (3 * hande_radius * hande_radius + coupler_shell_height * coupler_shell_height)}"
-                    ixy="0.0" ixz="0.0"
-                    iyy="${0.0833333 * coupler_mass * (3 * hande_radius * hande_radius + coupler_shell_height * coupler_shell_height)}"
-                    iyz="0.0"
-                    izz="${0.5 * coupler_mass * hande_radius * hande_radius}" />
-            </inertial>
-        </link>
         <!-- Gripper body -->
         <joint name="${prefix}robotiq_hande_base_joint" type="fixed">
-            <origin xyz="0 0 ${coupler_height}" rpy="0 0 0" />
-            <parent link="${prefix}robotiq_hande_coupler" />
+            <parent link="${parent}" />
             <child link="${prefix}robotiq_hande_link" />
+            <xacro:insert_block name="origin" />
         </joint>
         <link name="${prefix}robotiq_hande_link">
@@ -92,7 +57,7 @@
             </visual>
             <collision>
-                <origin xyz="0 0 ${(hande_height + coupler_hande_cutoff + 0.005) / 2}" rpy="0 0 0" />
+                <origin xyz="0 0 ${(hande_height + 0.005) / 2}" rpy="0 0 0" />
                 <geometry>
-                    <cylinder length="${hande_height + coupler_hande_cutoff + 0.005}" radius="${hande_radius + 0.001}" />
+                    <cylinder length="${hande_height + 0.005}" radius="${hande_radius + 0.001}" />
                 </geometry>
             </collision>

Commit message: Fixed Robotiq HandE finger value direction in URDF

File: robotiq_description/urdf/robotiq_hande_macro.urdf.xacro (robot description, xacro)
@@ -75,8 +75,8 @@
         <!-- Left finger (primary actuated joint) -->
         <joint name="${prefix}robotiq_hande_left_finger_joint" type="prismatic">
-            <origin xyz="0 0 ${hande_height}" rpy="0 0 0" />
+            <origin xyz="${gripper_closed_position} 0 ${hande_height}" rpy="0 0 0" />
             <parent link="${prefix}robotiq_hande_link" />
             <child link="${prefix}robotiq_hande_left_finger" />
-            <axis xyz="1 0 0" />
+            <axis xyz="-1 0 0" />
             <limit effort="130" lower="0.0" upper="${gripper_closed_position}" velocity="0.15" />
         </joint>
@@ -102,8 +102,8 @@
         <!-- Right finger (mimic of left) -->
         <joint name="${prefix}robotiq_hande_right_finger_joint" type="prismatic">
-            <origin xyz="0 0 ${hande_height}" rpy="0 0 0" />
+            <origin xyz="-${gripper_closed_position} 0 ${hande_height}" rpy="0 0 0" />
             <parent link="${prefix}robotiq_hande_link" />
             <child link="${prefix}robotiq_hande_right_finger" />
-            <axis xyz="-1 0 0" />
+            <axis xyz="1 0 0" />
             <limit effort="130" lower="0.0" upper="${gripper_closed_position}" velocity="0.15" />
             <mimic joint="${prefix}robotiq_hande_left_finger_joint" multiplier="1" offset="0" />
